File: kicad/ltl.kicad_sch (KiCad schematic)
At the start: 34 parts, among them J1 CONN_01X03, Q1 RUM001L02T2CL, Q2 RZM001P02T2L, U1 TPL5111, U2 ESP-12E, U3 DS18B20, U4 TPS73733DCQR

Commit message: Lots of added features and bug fixes
Parts:
- removed J1: CONN_01X03, Connector_JST:JST_XH_B3B-XH-A_1x03_P2.50mm_Vertical, symbol ltl-rescue:CONN_01X03
- added C10, C11, C12: 10uF, Capacitor_SMD:C_1206_3216Metric, symbol Device:C
- added D1: BAT54J, Diode_SMD:D_SOD-323F, symbol Diode:BAT54J
- added J1: Conn_01x06, Connector_PinHeader_2.54mm:PinHeader_1x06_P2.54mm_Horizontal, symbol Connector_Generic:Conn_01x06
- added Q3: BC857, Package_TO_SOT_SMD:SOT-23, symbol Transistor_BJT:BC857
- added R16, R17: 100, Resistor_SMD:R_1206_3216Metric, symbol ltl-rescue:R
- added R18: 10k, Resistor_SMD:R_1206_3216Metric, symbol ltl-rescue:R
- C1, C2, C3, C4, C5, C6, C7, C8, C9: footprint (none) -> Capacitor_SMD:C_1206_3216Metric
- R1, R10, R11, R12, R13, R14, R15, R2, R3, R4, R6, R7, R8, R9: footprint Resistor_THT:R_Axial_DIN0207_L6.3mm_D2.5mm_P10.16mm_Horizontal -> Resistor_SMD:R_1206_3216Metric
- R5: value 2,2k -> 10k; footprint Resistor_THT:R_Axial_DIN0207_L6.3mm_D2.5mm_P10.16mm_Horizontal -> Resistor_SMD:R_1206_3216Metric
- U3: footprint Package_TO_SOT_THT:TO-92 -> TO_SOT_Packages_THT:TO-92_Inline_Narrow_Oval
Connections:
- net +3V3: now also R5.1, U4.2 (OUT), C11.2, R18.2; no longer U2.3 (CH_PD), U4.5 (OUT)
- net BAT_DIV: now also U2.2 (ADC)
- net DONE: now also U2.10 (GPIO15)
- net DRIVE: now also U4.5 (EN); no longer U4.3 (EN)
- net GND: now also U4.3 (GND), C12.1, J1.5 (Pin_5), R17.1; no longer R5.1, U4.2 (GND)
- net RxD: now also J1.3 (Pin_3)
- net TxD: now also J1.2 (Pin_2)
- net RESET: now reaches R1.2, Reset1.1, U2.1 (REST)
- net RESET: now also C10.2; no longer U2.4 (GPIO16)
- net GPIO0: now reaches R3.1, U2.12 (GPIO0)
- net GPIO0: now also Q3.2 (E)
- net at R5.2: now also U2.3 (CH_PD); no longer U2.10 (GPIO15)
- net at R4.2, U3.2 (DQ): now also U2.13 (GPIO4); no longer U2.14 (GPIO5)
- new net: C11.1, Q3.3 (C), R17.2
- new net: D1.2 (A), R16.1
- new net: C12.2, Q3.1 (B), R16.2, R18.1
- new net DTR: C10.1, D1.1 (K), J1.1 (Pin_1)
Other:
- note added: "1"
- note added: "10"
- note added: "11"
- note added: "12"
- note added: "13"
- note added: "14"
- note added: "15"
- note added: "16"
- note added: "17"
- note added: "18"
- note added: "19"
- note added: "2"
- note added: "20"
- note added: "21"
- note added: "22"
- note added: "3"
- note added: "4"
- note added: "5"
- note added: "6"
- note added: "7"
- note added: "8"
- note added: "9"
- note added: "ADC"
- note added: "CH_EN"
- note added: "GND"
- note added: "GPIO0"
- note added: "GPIO1 U0TXD"
- note added: "GPIO10"
- note added: "GPIO11"
- note added: "GPIO12"
- note added: "GPIO13"
- note added: "GPIO14"
- note added: "GPIO15"
- note added: "GPIO16"
- note added: "GPIO2"
- note added: "GPIO3 U0RXD"
- note added: "GPIO4"
- note added: "GPIO5"
- note added: "GPIO6"
- note added: "GPIO7"
- note added: "GPIO8"
- note added: "GPIO9"
- note added: "RST"
- note added: "VCC"
- moved on the sheet: C1, C3, C5, C6, C7, C8, C9, Flash1, R1, R2, R3, R4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
